Commit message: Add kinematic solvers and interactive marker functionality
- Added forward kinematics query (fk_query.py)
- Added inverse kinematics solver (ik_solver.py)
- Added interactive target marker (interactive_target_marker.py)
- Added RViz configuration files
- Updated setup.py and PSM base URDF configuration

File: urdf/psm.base.xacro (robot description, xacro)
@@ -50,4 +50,11 @@
             </collision>
         </link>
+        <!-- Virtual tip for IK targeting -->
+        <link name="${prefix}_tool_virtual_tip"/>
+        <joint name="${prefix}_virtual_tip_dummy" type="fixed">
+          <parent link="${prefix}_tool_main_link"/>
+          <child link="${prefix}_tool_virtual_tip"/>
+          <origin xyz="0 0 0.4152" rpy="0 0 0"/>
+        </joint>
         <!-- Joint: Outer Roll Joint: Main to Wrist -->
         <joint name="${prefix}_outer_roll" type="revolute">
